File: preamp.kicad_pcb (KiCad board)
At the start: 2 copper layers, 117.1 x 47.1 mm, 37 parts, among them J1 Neck, J2 Bridge, J3 9V, J4 TRS, J5 Bridge GND, P1 Volume 250k log, P2 Hi Cut 250k log, P3 Bass Cut 1M, U1 LM4250

Commit message: cleaned up Fab layers
Parts:
- C1, C8: value C_Polarized 10uF -> 10uF
- C10, C6: value 1n -> 1nF
- C11: value 2,2n -> 2,2nF
- C2: value 220p -> 220pF
- C3: value 220p ( originally 200p) -> 220pF
- C4, C7: value 47n -> 47nF
- C5: value 10n -> 10nF
- C9: value 15n -> 15nF
